File: pcb/_autosave-SATS.kicad_sch (KiCad schematic)
At the start: 3 parts, among them J1 Raspberry_Pi_2_3, U1 MCP23017_SP, U2 MCP23017_SP

Commit message: Starting Parts Collection
Parts:
- added D?: 1N4007, Diode_THT:D_DO-41_SOD81_P10.16mm_Horizontal, symbol Diode:1N4007
- added U3: CD40109BE, DIP794W45P254L1969H508Q16, symbol CD40109BE:CD40109BE
Changed lines of the file:
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@@
 (kicad_sch (version 20211123) (generator eeschema)
   (paper "A4")
+  (symbol (lib_id "Diode:1N4007") (at 137.795 88.9 0) (unit 1)
+    (in_bom yes) (on_board yes) (fields_autoplaced)
+    (property "Reference" "D?" (id 0) (at 137.795 82.55 0))
+    (property "Value" "1N4007" (id 1) (at 137.795 85.09 0))
+    (property "Footprint" "Diode_THT:D_DO-41_SOD81_P10.16mm_Horizontal" (id 2) (at 137.795 93.345 0)
+      (effects (font (size 1.27 1.27)) hide)
+    )
+    (property "Datasheet" "http://www.vishay.com/docs/88503/1n4001.pdf" (id 3) (at 137.795 88.9 0)
+      (effects (font (size 1.27 1.27)) hide)
+    )
+    (pin "1")
+    (pin "2")
+  )
+  (symbol (lib_id "CD40109BE:CD40109BE") (at 126.365 156.21 0) (unit 1)
+    (in_bom yes) (on_board yes) (fields_autoplaced)
+    (property "Reference" "U3" (id 0) (at 126.365 130.81 0))
+    (property "Value" "CD40109BE" (id 1) (at 126.365 133.35 0))
+    (property "Footprint" "DIP794W45P254L1969H508Q16" (id 2) (at 126.365 156.21 0)
+      (effects (font (size 1.27 1.27)) (justify bottom) hide)
+    )
+    (property "Datasheet" "" (id 3) (at 126.365 156.21 0)
+      (effects (font (size 1.27 1.27)) hide)
+    )
+    (pin "1")
+    (pin "10")
+    (pin "11")
+    (pin "13")
+    (pin "14")
+    (pin "15")
+    (pin "16")
+    (pin "2")
+    (pin "3")
+    (pin "4")
+    (pin "5")
+    (pin "6")
+    (pin "7")
+    (pin "8")
+    (pin "9")
+  )
   (symbol (lib_id "Interface_Expansion:MCP23017_SP") (at 204.47 57.785 0) (unit 1)
     (in_bom yes) (on_board yes) (fields_autoplaced)
@@
   )
   (symbol_instances
+    (path "/10ba1107-77c4-4d57-9ffa-56a66acd4eae"
+      (reference "D?") (unit 1) (value "1N4007") (footprint "Diode_THT:D_DO-41_SOD81_P10.16mm_Horizontal")
+    )
     (path "/422a914e-8b99-4ff0-8ddf-1d6a3d23d7a7"
       (reference "J1") (unit 1) (value "Raspberry_Pi_2_3") (footprint "Connector_PinSocket_2.54mm:PinSocket_2x20_P2.54mm_Vertical")
@@
       (reference "U2") (unit 1) (value "MCP23017_SP") (footprint "Package_DIP:DIP-28_W7.62mm")
     )
-  )
+    (path "/201bf6e5-0ee1-4b89-8a4a-ce5cd24fad2f"
+      (reference "U3") (unit 1) (value "CD40109BE") (footprint "DIP794W45P254L1969H508Q16")
+    )
+  )
